File: hardware/driver.kicad_pcb (KiCad board)
At the start: 2 copper layers, 136 x 52 mm, 113 parts, among them J1 FPC16, J10 STEPPER0, J11 STEPPER7, J12 STEPPER6, J13 TEMP2, J14 I2C, J15 HEAT1, J16 TOOLSET, J17 HEAT2, J18 STEPPER1, J19 STEPPER3, J2 POWER, J20 AUX0, J21 XMIN, J22 XMAX, J23 AUX1, J24 YMIN, J25 YMAX, J26 AUX2, J27 STEPPER2, J28 STEPPER4, J29 ZMIN, J3 D/A, J30 ZMAX, J31 AUX3, J4 TEMP1, J5 BEDTEMP, J6 BED, J7 STEPPER5, J8 VDRV, J9 FAN, Q1 75N75, Q2 75N75, Q3 50N06, Q4 50N06, Q5 50N06, Q6 75N75, Q7 75N75, SW1 SW_DIP_x03, SW2 SW_DIP_x03, SW3 SW_DIP_x03, SW4 SW_DIP_x03, SW5 SW_DIP_x03, U1 74HC595, U10 A4988, U11 A4988, U12 TLP521, U13 TLP521, U14 TLP521, U15 TLP521, U2 AP1117-33, U3 XL2001, U4 74HC595, U5 MCP23017_SS, U6 74HC273, U7 A4988, U8 A4988, U9 A4988

Commit message: Add comment words on driver pcb silk layer
Signed-off-by: m24h <jjkkxyz@hotmail.com>
Other:
- board text added: "+ -"
- board text added: "AUX0"
- board text added: "AUX1"
- board text added: "AUX2"
- board text added: "AUX3"
- board text added: "BED"
- board text added: "BEDTEMP"
- board text added: "D/A"
- board text added: "FAN"
- board text added: "HEAT1"
- board text added: "HEAT2"
- board text added: "I2C"
- board text added: "MS1 MS2 MS3"
- board text added: "POWER"
- board text added: "STEPPER0"
- board text added: "STEPPER1"
- board text added: "STEPPER2"
- board text added: "STEPPER3"
- board text added: "STEPPER4"
- board text added: "STEPPER5"
- board text added: "STEPPER6"
- board text added: "STEPPER7"
- board text added: "TEMP1"
- board text added: "TEMP2"
- board text added: "TOOLSET"
- board text added: "VDRV"
- board text added: "XMAX"
- board text added: "XMIN"
- board text added: "YMAX"
- board text added: "YMIN"
- board text added: "ZMAX"
- board text added: "ZMIN"
Changed lines of the file:
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@@
   (general
     (thickness 1.6)
-    (drawings 49)
+    (drawings 96)
     (tracks 1521)
     (zones 0)
@@
     (descr "Through hole straight pin header, 1x02, 2.54mm pitch, single row")
     (tags "Through hole pin header THT 1x02 2.54mm single row")
-    (fp_text reference J4 (at 0 2.33 180) (layer B.SilkS)
+    (fp_text reference J4 (at 1.6711 -0.4301 180) (layer B.SilkS)
       (effects (font (size 1 1) (thickness 0.15)) (justify mirror))
     )
@@
     (descr "Through hole straight pin header, 1x04, 2.54mm pitch, single row")
     (tags "Through hole pin header THT 1x04 2.54mm single row")
-    (fp_text reference J14 (at 0 2.33 270) (layer B.SilkS)
+    (fp_text reference J14 (at -0.1535 -10.2977 270) (layer B.SilkS)
       (effects (font (size 1 1) (thickness 0.15)) (justify mirror))
     )
@@
     (descr "Through hole straight pin header, 1x03, 2.54mm pitch, single row")
     (tags "Through hole pin header THT 1x03 2.54mm single row")
-    (fp_text reference J21 (at 0 2.33 270) (layer B.SilkS)
+    (fp_text reference J21 (at 0.3 7.02 270) (layer B.SilkS)
       (effects (font (size 1 1) (thickness 0.15)) (justify mirror))
     )
@@
     (descr "Through hole straight pin header, 1x03, 2.54mm pitch, single row")
     (tags "Through hole pin header THT 1x03 2.54mm single row")
-    (fp_text reference J22 (at 0 2.33 270) (layer B.SilkS)
+    (fp_text reference J22 (at 0.2 7.02 270) (layer B.SilkS)
       (effects (font (size 1 1) (thickness 0.15)) (justify mirror))
     )
@@
     (descr "Through hole straight pin header, 1x03, 2.54mm pitch, single row")
     (tags "Through hole pin header THT 1x03 2.54mm single row")
-    (fp_text reference J24 (at 0 2.33 270) (layer B.SilkS)
+    (fp_text reference J24 (at 0.1 6.82 270) (layer B.SilkS)
       (effects (font (size 1 1) (thickness 0.15)) (justify mirror))
     )
@@
     (descr "Through hole straight pin header, 1x03, 2.54mm pitch, single row")
     (tags "Through hole pin header THT 1x03 2.54mm single row")
-    (fp_text reference J25 (at 0 2.33 270) (layer B.SilkS)
+    (fp_text reference J25 (at 0.3 6.62 270) (layer B.SilkS)
       (effects (font (size 1 1) (thickness 0.15)) (justify mirror))
     )
@@
       (effects (font (size 1 1) (thickness 0.15)) (justify mirror))
     )
-    (fp_text value STEPPER4 (at -2.7801 -4.1638 180) (layer B.Fab)
+    (fp_text value STEPPER4 (at -2.6801 -4.1638 180) (layer B.Fab)
       (effects (font (size 1 1) (thickness 0.15)) (justify mirror))
     )
@@
     (descr "Through hole straight pin header, 1x03, 2.54mm pitch, single row")
     (tags "Through hole pin header THT 1x03 2.54mm single row")
-    (fp_text reference J29 (at 0 2.33 270) (layer B.SilkS)
+    (fp_text reference J29 (at 0 6.72 270) (layer B.SilkS)
       (effects (font (size 1 1) (thickness 0.15)) (justify mirror))
     )
@@
     (descr "Through hole straight pin header, 1x03, 2.54mm pitch, single row")
     (tags "Through hole pin header THT 1x03 2.54mm single row")
-    (fp_text reference J30 (at 0 2.33 270) (layer B.SilkS)
+    (fp_text reference J30 (at -0.1 6.82 270) (layer B.SilkS)
       (effects (font (size 1 1) (thickness 0.15)) (justify mirror))
     )
@@
     )
   )
+  (gr_text "MS1\nMS2\nMS3" (at 213.3 64.7 90) (layer B.SilkS)
+    (effects (font (size 1 1) (thickness 0.15)) (justify mirror))
+  )
+  (gr_text "MS1\nMS2\nMS3" (at 148.6 88.9 90) (layer B.SilkS)
+    (effects (font (size 1 1) (thickness 0.15)) (justify mirror))
+  )
+  (gr_text "MS1\nMS2\nMS3" (at 170.2 89.5 90) (layer B.SilkS)
+    (effects (font (size 1 1) (thickness 0.15)) (justify mirror))
+  )
+  (gr_text "MS1\nMS2\nMS3" (at 191.5 89.5 90) (layer B.SilkS)
+    (effects (font (size 1 1) (thickness 0.15)) (justify mirror))
+  )
+  (gr_text "MS1\nMS2\nMS3" (at 213.3 89.5 90) (layer B.SilkS)
+    (effects (font (size 1 1) (thickness 0.15)) (justify mirror))
+  )
+  (gr_text "+     -" (at 94.4 73.8) (layer B.SilkS)
+    (effects (font (size 1 1) (thickness 0.15)) (justify mirror))
+  )
+  (gr_text "+     -" (at 94.9 56.2) (layer B.SilkS)
+    (effects (font (size 1 1) (thickness 0.15)) (justify mirror))
+  )
+  (gr_text "+\n-" (at 87.4 63.5 270) (layer B.SilkS)
+    (effects (font (size 1 1) (thickness 0.15)) (justify mirror))
+  )
+  (gr_text VDRV (at 87.4 60.7 270) (layer B.SilkS)
+    (effects (font (size 1 1) (thickness 0.15)) (justify mirror))
+  )
+  (gr_text "+\n-" (at 87.3 72.8 270) (layer B.SilkS)
+    (effects (font (size 1 1) (thickness 0.15)) (justify mirror))
+  )
+  (gr_text POWER (at 87.4 69.3 270) (layer B.SilkS)
+    (effects (font (size 1 1) (thickness 0.15)) (justify mirror))
+  )
+  (gr_text - (at 125.4 105.4) (layer B.SilkS)
+    (effects (font (size 1 1) (thickness 0.15)) (justify mirror))
+  )
+  (gr_text + (at 130.4 105.4) (layer B.SilkS)
+    (effects (font (size 1 1) (thickness 0.15)) (justify mirror))
+  )
+  (gr_text - (at 113.6 105.5) (layer B.SilkS)
+    (effects (font (size 1 1) (thickness 0.15)) (justify mirror))
+  )
+  (gr_text + (at 119.6 105.5) (layer B.SilkS)
+    (effects (font (size 1 1) (thickness 0.15)) (justify mirror))
+  )
+  (gr_text - (at 102.8 105.5) (layer B.SilkS)
+    (effects (font (size 1 1) (thickness 0.15)) (justify mirror))
+  )
+  (gr_text + (at 108.6 105.5) (layer B.SilkS)
+    (effects (font (size 1 1) (thickness 0.15)) (justify mirror))
+  )
+  (gr_text - (at 91.9 105.5) (layer B.SilkS)
+    (effects (font (size 1 1) (thickness 0.15)) (justify mirror))
+  )
+  (gr_text + (at 96.9 105.5) (layer B.SilkS)
+    (effects (font (size 1 1) (thickness 0.15)) (justify mirror))
+  )
+  (gr_text BED (at 94.5 105.6) (layer B.SilkS)
+    (effects (font (size 1 1) (thickness 0.15)) (justify mirror))
+  )
+  (gr_text HEAT1 (at 105.7 105.6) (layer B.SilkS)
+    (effects (font (size 1 1) (thickness 0.15)) (justify mirror))
+  )
+  (gr_text HEAT2 (at 116.7 105.6) (layer B.SilkS)
+    (effects (font (size 1 1) (thickness 0.15)) (justify mirror))
+  )
+  (gr_text FAN (at 127.8 105.5) (layer B.SilkS)
+    (effects (font (size 1 1) (thickness 0.15)) (justify mirror))
+  )
+  (gr_text TOOLSET (at 155.2 68.2) (layer B.SilkS)
+    (effects (font (size 1 1) (thickness 0.15)) (justify mirror))
+  )
+  (gr_text I2C (at 160.4 76.6) (layer B.SilkS)
+    (effects (font (size 1 1) (thickness 0.15)) (justify mirror))
+  )
+  (gr_text ZMAX (at 129.6 77.6) (layer B.SilkS)
+    (effects (font (size 1 1) (thickness 0.15)) (justify mirror))
+  )
+  (gr_text ZMIN (at 129.8 73.7) (layer B.SilkS)
+    (effects (font (size 1 1) (thickness 0.15)) (justify mirror))
+  )
+  (gr_text YMAX (at 129.8 70.1) (layer B.SilkS)
+    (effects (font (size 1 1) (thickness 0.15)) (justify mirror))
+  )
+  (gr_text YMIN (at 129.8 66.2) (layer B.SilkS)
+    (effects (font (size 1 1) (thickness 0.15)) (justify mirror))
+  )
+  (gr_text XMAX (at 129.6 62) (layer B.SilkS)
+    (effects (font (size 1 1) (thickness 0.15)) (justify mirror))
+  )
+  (gr_text XMIN (at 129.6 58) (layer B.SilkS)
+    (effects (font (size 1 1) (thickness 0.15)) (justify mirror))
+  )
+  (gr_text AUX0 (at 151.6 78.2) (layer B.SilkS)
+    (effects (font (size 1 1) (thickness 0.15)) (justify mirror))
+  )
+  (gr_text AUX1 (at 153 74.2) (layer B.SilkS)
+    (effects (font (size 1 1) (thickness 0.15)) (justify mirror))
+  )
+  (gr_text AUX2 (at 153 70.6) (layer B.SilkS)
+    (effects (font (size 1 1) (thickness 0.15)) (justify mirror))
+  )
+  (gr_text AUX3 (at 145.8 64.6) (layer B.SilkS)
+    (effects (font (size 1 1) (thickness 0.15)) (justify mirror))
+  )
+  (gr_text TEMP2 (at 143.5 62.5) (layer B.SilkS)
+    (effects (font (size 1 1) (thickness 0.15)) (justify mirror))
+  )
+  (gr_text TEMP1 (at 147.9 55.9) (layer B.SilkS)
+    (effects (font (size 1 1) (thickness 0.15)) (justify mirror))
+  )
+  (gr_text BEDTEMP (at 154.7 62.9) (layer B.SilkS)
+    (effects (font (size 1 1) (thickness 0.15)) (justify mirror))
+  )
+  (gr_text D/A (at 181.4 65.4) (layer B.SilkS)
+    (effects (font (size 1 1) (thickness 0.15)) (justify mirror))
+  )
+  (gr_text STEPPER5 (at 191 70.2) (layer B.SilkS)
+    (effects (font (size 1 1) (thickness 0.15)) (justify mirror))
+  )
+  (gr_text STEPPER6 (at 191 68.6) (layer B.SilkS)
+    (effects (font (size 1 1) (thickness 0.15)) (justify mirror))
+  )
+  (gr_text STEPPER7 (at 191 56.6) (layer B.SilkS)
+    (effects (font (size 1 1) (thickness 0.15)) (justify mirror))
+  )
+  (gr_text STEPPER0 (at 148.2 104.4) (layer B.SilkS)
+    (effects (font (size 1 1) (thickness 0.15)) (justify mirror))
+  )
+  (gr_text STEPPER1 (at 169.4 104.4) (layer B.SilkS)
+    (effects (font (size 1 1) (thickness 0.15)) (justify mirror))
+  )
+  (gr_text STEPPER2 (at 190.6 104.4) (layer B.SilkS)
+    (effects (font (size 1 1) (thickness 0.15)) (justify mirror))
+  )
+  (gr_text STEPPER3 (at 212.4 104.4) (layer B.SilkS)
+    (effects (font (size 1 1) (thickness 0.15)) (justify mirror))
+  )
+  (gr_text STEPPER4 (at 212.3 79.7) (layer B.SilkS)
+    (effects (font (size 1 1) (thickness 0.15)) (justify mirror))
+  )
   (gr_text - (at 92 73.9) (layer B.Fab)
